File: PCB/shield_Respirador/shield_Respirador.sch (KiCad schematic (older format))
At the start: 30 parts, among them P1 Digital, P10 CONN_01X01, P11 CONN_01X01, P12 CONN_01X01, P13 CONN_01X01, P2 Power, P3 Analog, P4 Analog, P5 PWM, P6 PWM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

Commit message: version 0.4
Parts:
- added Alarma_Sonido1: Buzzer, Buzzer_Beeper:MagneticBuzzer_ProSignal_ABI-009-RC, symbol Device:Buzzer
- added Drivermotor1: Pololu_Breakout_DRV8825, Module:Pololu_Breakout-16_15.2x20.3mm, symbol Driver_Motor:Pololu_Breakout_DRV8825
- added Final_De_Carrera1: Conn_01x03_Female, Connector_PinSocket_2.00mm:PinSocket_1x03_P2.00mm_Vertical, symbol Connector:Conn_01x03_Female
- added R_Buzzer1: 220, Resistor_THT:R_Axial_DIN0207_L6.3mm_D2.5mm_P10.16mm_Horizontal, symbol Device:R
- added Sensor_Presion1: MPXA6115A, Package_DIP:DIP-8_W7.62mm_LongPads, symbol Sensor_Pressure:MPXA6115A
- added Set_configuracion1: SW_Push, TerminalBlock:TerminalBlock_bornier-2_P5.08mm, symbol Switch:SW_Push
- added Toogle_configuracion1: SW_Push_SPDT, TerminalBlock:TerminalBlock_bornier-3_P5.08mm, symbol Switch:SW_Push_SPDT
- added conector_motor1: Conn_01x04_Female, Connector_PinSocket_2.00mm:PinSocket_1x04_P2.00mm_Vertical, symbol Connector:Conn_01x04_Female
- On/off1: footprint Connector:Banana_Jack_3Pin -> TerminalBlock:TerminalBlock_bornier-3_P5.08mm
Connections:
- net 31: now also R_Buzzer1.1
- net GND: now also Alarma_Sonido1.2 (+)
- new net: Alarma_Sonido1.1 (-), R_Buzzer1.2
Other:
- moved on the sheet: C_1, C_2, LCD1, On/off1A, R_Alarma1, R_Alarma2, R_Alarma3, R_configuracion1, Regulador-12V-5V1, jack_12V1

Commit message: version 0.41 Esquematico terminado y irganizado
Parts:
- added R1: R, symbol Device:R
- added R_Configuración: 220, symbol Device:R
- Drivermotor1: value Pololu_Breakout_DRV8825 -> DRV8825
- renumbered Toogle_configuracion1 to Toogle_configuracion
Connections:
- net +12V: now also Drivermotor1.8 (VMOT)
- net +5V: now also Final_De_Carrera1.1 (Pin_1), P_Frecuencia1.3, P_Presion1.3, P_volumen_tidal1.3, Sensor_Presion1.2 (Vcc), Set_configuracion1.2, Toogle_configuracion.2 (B)
- net 10(**): now also Drivermotor1.13 (~RST)
- net 11(**): now also Drivermotor1.14 (~SLP)
- net 29: now also Final_De_Carrera1.2 (Pin_2)
- net 42: now also Toogle_configuracion.3 (C), R_Configuración.1
- net 43: now also Set_configuracion1.1, R1.1
- net 8(**): now also Drivermotor1.16 (DIR)
- net 9(**): now also Drivermotor1.15 (STEP)
- net A8: now also Sensor_Presion1.4 (Vout)
- net GND: now also Drivermotor1.1 (GND), Drivermotor1.7 (GND), Final_De_Carrera1.3 (Pin_3), P_Frecuencia1.1, P_Presion1.1, P_volumen_tidal1.1, Sensor_Presion1.3 (GND), R1.2, R_Configuración.2
- net at Drivermotor1.3 (A2): now also conector_motor1.2 (Pin_2)
- net at Drivermotor1.4 (A1): now also conector_motor1.1 (Pin_1)
- net at Drivermotor1.5 (B1): now also conector_motor1.3 (Pin_3)
- net at Drivermotor1.6 (B2): now also conector_motor1.4 (Pin_4)
Other:
- note added: "Alimentación 12 V y 5V\n"
- note added: "Botones de configuracion\n"
- note added: "Driver y servomotor\n"
- note added: "Indicadores y alarmas"
- note added: "Sensor presion y final de carrera\n"
- note added: "Sistema de visualización (LCD)\n"
- moved on the sheet: C_1, C_2, Drivermotor1, Final_De_Carrera1, LCD1, On/off1A, P_Frecuencia1, P_Presion1, P_volumen_tidal1, Regulador-12V-5V1, Sensor_Presion1, Set_configuracion1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

Commit message: version 0.5 se termina esquematico y renderizacion
Parts:
- added P14, P15, P16, P17, P18, P19: CONN_01X01, Socket_Arduino_Mega:Arduino_1pin, symbol Connector_Generic:Conn_01x01
- R1: footprint (none) -> Resistor_THT:R_Axial_DIN0207_L6.3mm_D2.5mm_P10.16mm_Horizontal
- R_Configuración1: renamed from R_Configuración; footprint (none) -> Resistor_THT:R_Axial_DIN0207_L6.3mm_D2.5mm_P10.16mm_Horizontal
- renumbered Toogle_configuracion to Toogle_configuracion1
Connections:
- net 20(SDA): now also LCD1.4 (RS)
- net 21(SCL): now also LCD1.3 (VO)
- net 22: now also R_Buzzer1.1
- net 29: no longer Final_De_Carrera1.2 (Pin_2)
- net 30: now also R1.1, Set_configuracion1.1
- net 31: no longer R_Buzzer1.1
- net 43: no longer R1.1, Set_configuracion1.1
- net 49: now also Final_De_Carrera1.2 (Pin_2)
- net SCL: no longer LCD1.5 (R/W)
- net SDA: no longer LCD1.6 (E)
- no-connect marks 7 -> 13
Other:
- note added: "Huecos de sujecion\n"
Changed lines of the file:
@@
 Wire Wire Line
 	4600 1600 4700 1600
-Text Label 3200 2000 3    60   ~ 0
-SDA
-Text Label 3300 2000 3    60   ~ 0
-SCL
 $Comp
 L Device:LED D1
@@
 	7300 1750 7500 1750
 Text Label 6700 1750 0    60   ~ 0
-31
+22
 $Comp
 L power:GND #PWR0109
@@
 $EndComp
 $Comp
-L Switch:SW_Push_SPDT Toogle_configuracion
+L Switch:SW_Push_SPDT Toogle_configuracion1
 U 1 1 5E9ACB74
 P 2100 4600
-F 0 "Toogle_configuracion" H 2550 4800 50  0000 C CNN
+F 0 "Toogle_configuracion1" H 2550 4800 50  0000 C CNN
 F 1 "SW_Push_SPDT" H 2100 4794 50  0001 C CNN
 F 2 "TerminalBlock:TerminalBlock_bornier-3_P5.08mm" H 2100 4600 50  0001 C CNN
@@
 F 0 "R1" H 2320 3896 50  0000 L CNN
 F 1 "R" H 2320 3805 50  0000 L CNN
-F 2 "" V 2180 3850 50  0001 C CNN
+F 2 "Resistor_THT:R_Axial_DIN0207_L6.3mm_D2.5mm_P10.16mm_Horizontal" V 2180 3850 50  0001 C CNN
 F 3 "~" H 2250 3850 50  0001 C CNN
 	1    2250 3850
@@
 	500  500  8350 500
 $Comp
-L power:GND #PWR?
+L power:GND #PWR0112
 U 1 1 5EBB921E
 P 4350 4900
-F 0 "#PWR?" H 4350 4650 50  0001 C CNN
+F 0 "#PWR0112" H 4350 4650 50  0001 C CNN
 F 1 "GND" H 4355 4727 50  0000 C CNN
 F 2 "" H 4350 4900 50  0001 C CNN
@@
 	4900 4350 4900 4300
 $Comp
-L power:+12V #PWR?
+L power:+12V #PWR0113
 U 1 1 5EBFCEF3
 P 4350 3450
-F 0 "#PWR?" H 4350 3300 50  0001 C CNN
+F 0 "#PWR0113" H 4350 3300 50  0001 C CNN
 F 1 "+12V" H 4365 3623 50  0000 C CNN
 F 2 "" H 4350 3450 50  0001 C CNN
@@
 8(**)
 $Comp
-L power:+5V #PWR?
+L power:+5V #PWR0114
 U 1 1 5EC6C8DF
 P 7250 3400
-F 0 "#PWR?" H 7250 3250 50  0001 C CNN
+F 0 "#PWR0114" H 7250 3250 50  0001 C CNN
 F 1 "+5V" H 7265 3573 50  0000 C CNN
 F 2 "" H 7250 3400 50  0001 C CNN
@@
 $EndComp
 $Comp
-L power:GND #PWR?
+L power:GND #PWR0115
 U 1 1 5EC6D60F
 P 7250 4000
-F 0 "#PWR?" H 7250 3750 50  0001 C CNN
+F 0 "#PWR0115" H 7250 3750 50  0001 C CNN
 F 1 "GND" H 7255 3827 50  0000 C CNN
 F 2 "" H 7250 4000 50  0001 C CNN
@@
 A8
 Text Label 6850 4750 2    60   ~ 0
-29
-$Comp
-L power:+5V #PWR?
+49
+$Comp
+L power:+5V #PWR0116
 U 1 1 5ECD86AB
 P 6850 4650
-F 0 "#PWR?" H 6850 4500 50  0001 C CNN
+F 0 "#PWR0116" H 6850 4500 50  0001 C CNN
 F 1 "+5V" H 6865 4823 50  0000 C CNN
 F 2 "" H 6850 4650 50  0001 C CNN
@@
 $EndComp
 $Comp
-L power:GND #PWR?
+L power:GND #PWR0117
 U 1 1 5ECD8EB5
 P 6850 4850
-F 0 "#PWR?" H 6850 4600 50  0001 C CNN
+F 0 "#PWR0117" H 6850 4600 50  0001 C CNN
 F 1 "GND" H 6855 4677 50  0000 C CNN
 F 2 "" H 6850 4850 50  0001 C CNN
@@
 $EndComp
 $Comp
-L Device:R R_Configuración
+L Device:R R_Configuración1
 U 1 1 5ECDBE87
 P 2300 4850
-F 0 "R_Configuración" H 2370 4896 50  0000 L CNN
+F 0 "R_Configuración1" H 2370 4896 50  0000 L CNN
 F 1 "220" H 2370 4805 50  0000 L CNN
-F 2 "" V 2230 4850 50  0001 C CNN
+F 2 "Resistor_THT:R_Axial_DIN0207_L6.3mm_D2.5mm_P10.16mm_Horizontal" V 2230 4850 50  0001 C CNN
 F 3 "~" H 2300 4850 50  0001 C CNN
 	1    2300 4850
@@
 $EndComp
 $Comp
-L power:GND #PWR?
+L power:GND #PWR0118
 U 1 1 5ECE4317
 P 2300 5000
-F 0 "#PWR?" H 2300 4750 50  0001 C CNN
+F 0 "#PWR0118" H 2300 4750 50  0001 C CNN
 F 1 "GND" H 2305 4827 50  0000 C CNN
 F 2 "" H 2300 5000 50  0001 C CNN
@@
 $EndComp
 $Comp
-L power:+5V #PWR?
+L power:+5V #PWR0119
 U 1 1 5ECE4A68
 P 1900 4600
-F 0 "#PWR?" H 1900 4450 50  0001 C CNN
+F 0 "#PWR0119" H 1900 4450 50  0001 C CNN
 F 1 "+5V" H 1915 4773 50  0000 C CNN
 F 2 "" H 1900 4600 50  0001 C CNN
@@
 	3500 2950 5000 2950
 $Comp
-L power:GND #PWR?
+L power:GND #PWR0120
 U 1 1 5EDCBFC1
 P 2250 4000
-F 0 "#PWR?" H 2250 3750 50  0001 C CNN
+F 0 "#PWR0120" H 2250 3750 50  0001 C CNN
 F 1 "GND" H 2255 3827 50  0000 C CNN
 F 2 "" H 2250 4000 50  0001 C CNN
@@
 $EndComp
 Text Label 1900 3700 0    60   ~ 0
-43
+30
 Wire Wire Line
 	1900 3700 2250 3700
 Connection ~ 2250 3700
 $Comp
-L power:+5V #PWR?
+L power:+5V #PWR0121
 U 1 1 5EDECEA7
 P 2850 3700
-F 0 "#PWR?" H 2850 3550 50  0001 C CNN
+F 0 "#PWR0121" H 2850 3550 50  0001 C CNN
 F 1 "+5V" H 2865 3873 50  0000 C CNN
 F 2 "" H 2850 3700 50  0001 C CNN
@@
 Wire Notes Line
 	7600 2750 7600 2950
+Text Label 3400 2000 3    60   ~ 0
+20(SDA)
+Text Label 3200 1200 1    60   ~ 0
+21(SCL)
+$Comp
+L Connector_Generic:Conn_01x01 P14
+U 1 1 5EF71DAC
+P 7000 5900
+F 0 "P14" V 7100 5900 31  0000 C CNN
+F 1 "CONN_01X01" V 7100 5900 50  0001 C CNN
+F 2 "Socket_Arduino_Mega:Arduino_1pin" H 7000 5900 50  0001 C CNN
+F 3 "" H 7000 5900 50  0000 C CNN
+	1    7000 5900
+	0    -1   -1   0
+$EndComp
+$Comp
+L Connector_Generic:Conn_01x01 P15
+U 1 1 5EF71DB2
+P 7100 5900
+F 0 "P15" V 7200 5900 31  0000 C CNN
+F 1 "CONN_01X01" V 7200 5900 50  0001 C CNN
+F 2 "Socket_Arduino_Mega:Arduino_1pin" H 7100 5900 50  0001 C CNN
+F 3 "" H 7100 5900 50  0000 C CNN
+	1    7100 5900
+	0    -1   -1   0
+$EndComp
+$Comp
+L Connector_Generic:Conn_01x01 P16
+U 1 1 5EF71DB8
+P 7200 5900
+F 0 "P16" V 7300 5900 31  0000 C CNN
+F 1 "CONN_01X01" V 7300 5900 50  0001 C CNN
+F 2 "Socket_Arduino_Mega:Arduino_1pin" H 7200 5900 50  0001 C CNN
+F 3 "" H 7200 5900 50  0000 C CNN
+	1    7200 5900
+	0    -1   -1   0
+$EndComp
+$Comp
+L Connector_Generic:Conn_01x01 P17
+U 1 1 5EF71DBE
+P 7300 5900
+F 0 "P17" V 7400 5900 31  0000 C CNN
+F 1 "CONN_01X01" V 7400 5900 50  0001 C CNN
+F 2 "Socket_Arduino_Mega:Arduino_1pin" H 7300 5900 50  0001 C CNN
+F 3 "" H 7300 5900 50  0000 C CNN
+	1    7300 5900
+	0    -1   -1   0
+$EndComp
+$Comp
+L Connector_Generic:Conn_01x01 P18
+U 1 1 5EF71DC4
+P 7400 5900
+F 0 "P18" V 7500 5900 31  0000 C CNN
+F 1 "CONN_01X01" V 7500 5900 50  0001 C CNN
+F 2 "Socket_Arduino_Mega:Arduino_1pin" H 7400 5900 50  0001 C CNN
+F 3 "" H 7400 5900 50  0000 C CNN
+	1    7400 5900
+	0    -1   -1   0
+$EndComp
+$Comp
+L Connector_Generic:Conn_01x01 P19
+U 1 1 5EF71DCA
+P 7500 5900
+F 0 "P19" V 7600 5900 31  0000 C CNN
+F 1 "CONN_01X01" V 7600 5900 50  0001 C CNN
+F 2 "Socket_Arduino_Mega:Arduino_1pin" H 7500 5900 50  0001 C CNN
+F 3 "" H 7500 5900 50  0000 C CNN
+	1    7500 5900
+	0    -1   -1   0
+$EndComp
+NoConn ~ 7000 6100
+NoConn ~ 7100 6100
+NoConn ~ 7200 6100
+NoConn ~ 7300 6100
+NoConn ~ 7400 6100
+NoConn ~ 7500 6100
+Text Notes 6075 5475 0    60   ~ 0
+Huecos de sujecion\n
+Wire Notes Line
+	6050 5550 7650 5550
+Wire Notes Line
+	7650 5350 7650 5550
 $EndSCHEMATC
